Commit message: modified:   src/gcode_interpreter/scripts/main.py 	new file:   src/master_launch/master_connect.launch 	modified:   src/ur5_apla/urdf/printhead.xacro 	modified:   src/ur5_apla_moveit_config/scripts/singlePose.py

File: src/ur5_apla/urdf/printhead.xacro (robot description, xacro)
@@ -15,5 +15,5 @@
         <geometry>
           <!-- The path to the visual meshes in the package. This can be the dae variant -->
-          <mesh filename="package://ur5_apla/meshes/printhead/visual/printheadv2.stl"/>
+          <mesh filename="package://ur5_apla/meshes/printhead/visual/printheadv2.dae"/>
         </geometry>
       </visual>
@@ -21,5 +21,5 @@
         <geometry>
           <!-- The path to the collision meshes in the package. -->
-          <mesh filename="package://ur5_apla/meshes/printhead/collision/printheadv2.dae"/>
+          <mesh filename="package://ur5_apla/meshes/printhead/collision/printheadv2.stl"/>
         </geometry>
       </collision>
